File: LumioV2.kicad_sch (KiCad schematic)
At the start: 20 parts, among them J1 Raspi 5, J10 US Dist - Back, J2 I2C POINT 1 - QWIIC, J3 I2C POINT 2 - QWIIC, J4 I2C POINT 3 - JST-PH, J5 Display Connector, J6 MOTOR A, J7 MOTOR B, J8 I2C POINT 4 - JST-PH, J9 US Dist - Front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

Commit message: Added safety and pull circuit to the L298N block outputs
Parts:
- added D2, D3, D4, D5, D6, D7, D8, D9: 1N4148WT, Diode_SMD:D_SOD-523, symbol Diode:1N4148WT
Connections:
- net GND: now also U1.1 (SENSE_A), U1.15 (SENSE_B), D2.2 (A), D3.2 (A), D4.2 (A), D5.2 (A)
- net at J7.1 (Pin_1), U1.13 (OUT3): now also D4.1 (K), D8.2 (A)
- net at J7.2 (Pin_2), U1.14 (OUT4): now also D5.1 (K), D9.2 (A)
- net at J6.1 (Pin_1), U1.2 (OUT1): now also D2.1 (K), D6.2 (A)
- net at J6.2 (Pin_2), U1.3 (OUT2): now also D3.1 (K), D7.2 (A)
- net at C2.1, C5.2, D1.1 (K)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: now also D6.1 (K), D7.1 (K), D8.1 (K), D9.1 (K)
Other:
- note added: "L298N Motor Control Segment"
- moved on the sheet: J5
