File: LumioV2.kicad_sch (KiCad schematic)
At the start: 81 parts, among them J1 I2C POINT 1 - QWIIC, J10 MOTOR B, J11 Analog Input, J12 Analog Input, J13 Analog Input, J14 Analog Input, J15 Analog Input, J16 Analog Input, J17 Analog Input, J18 Analog Input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

Commit message: re-started routing, for clearer routes. also moved to dsi conenctor for display
Parts:
- removed C22, C23, C24: 100nF, Capacitor_SMD:C_0402_1005Metric_Pad0.74x0.62mm_HandSolder, symbol Device:C_Small
- removed J8: Display Connector, Connector_PinHeader_2.54mm:PinHeader_2x13_P2.54mm_Vertical, symbol Connector_Generic:Conn_02x13_Odd_Even
- removed P1: USB_C_Plug_USB2.0, Connector_USB:USB_C_Receptacle_GCT_USB4105-xx-A_16P_TopMnt_Horizontal, symbol Connector:USB_C_Plug_USB2.0
- removed R2: 5.1K, Resistor_SMD:R_0805_2012Metric_Pad1.20x1.40mm_HandSolder, symbol Device:R_Small
- added J8: USB_C_Receptacle_USB2.0_14P, Connector_USB:USB_C_Receptacle_Amphenol_12401610E4-2A, symbol Connector:USB_C_Receptacle_USB2.0_14P
- added R5, R6: 5.1K, Resistor_SMD:R_0805_2012Metric_Pad1.20x1.40mm_HandSolder, symbol Device:R_Small
- added Y2: ECS-2520MV-xxx-xx, Oscillator:Oscillator_SMD_ECS_2520MV-xxx-xx-4Pin_2.5x2.0mm, symbol Oscillator:ECS-2520MV-xxx-xx
- C5: footprint Capacitor_SMD:C_0402_1005Metric_Pad0.74x0.62mm_HandSolder -> Capacitor_SMD:C_1210_3225Metric
Connections:
- net +5V: now also J8.A4 (VBUS), J8.A9 (VBUS), J8.B4 (VBUS), J8.B9 (VBUS)
- net GND: now also J8.A1 (GND), J8.A12 (GND), J8.B1 (GND), J8.B12 (GND), J8.S1 (SHIELD), R5.2, R6.1
- net USB_N: now also J8.A7 (D-), J8.B7 (D-)
- net USB_P: now also J8.A6 (D+), J8.B6 (D+)
- net at J20.1 (Pin_1), U4.2 (GPIO0): now also J5.10 (Pin_10)
- net at J20.2 (Pin_2), U4.3 (GPIO1): now also J5.8 (Pin_8)
- new net: J8.A5 (CC1), R5.1
- new net: J8.B5 (CC2), R6.2
- no-connect marks 19 -> 0
