File: LumioV2.kicad_pcb (KiCad board)
At the start: 2 copper layers, 86 parts, among them J1 Raspi 5, J10 Analog Input, J11 Analog Input, J12 Analog Input, J13 Analog Input, J14 Analog Input, J15 Analog Input, J16 Analog Input, J17 Analog Input, J18 US Dist - Back, J19 US Dist - Front, J2 USB_C_Receptacle_USB2.0_14P, J20 Header programmer, J21 Conn_02x02_Odd_Even, J3 Conn_02x13_Odd_Even, J4 I2C POINT 4 - JST-PH, J5 I2C POINT 3 - JST-PH, J6 I2C POINT 2 - QWIIC, J7 I2C POINT 1 - QWIIC, J8 MOTOR B, J9 MOTOR A, SW1 SW_Push, SW2 SW_Push, U1 LM2577T-ADJ/NOPB, U2 L298N, U3 W25Q64JVXGIQ TR, U4 MCP3008, U5 RP2040, Y1 ECS-2520MV-xxx-xx

Commit message: finished routing, added 3d files for most parts
Parts:
- removed the C17 at (253.8, 122.7)
- removed the C18 at (257.0, 134.5)
- removed the C19 at (260.2, 126.6)
- removed the C21 at (260.2, 122.7)
- removed the C22 at (260.2, 128.6)
- removed the C24 at (257.0, 128.6)
- removed the C26 at (253.8, 120.7)
- removed the C28 at (260.2, 120.7)
- removed the C29 at (257.0, 130.6)
- removed the C31 at (257.0, 132.6)
- removed C35: 100nF, Capacitor_SMD:C_0402_1005Metric_Pad0.74x0.62mm_HandSolder
- removed the R1 at (136.6, 51.5)
- removed the R2 at (139.5, 51.5)
- removed the U3 at (89.4, 135.3)
- added C13: 1uF, Capacitor_SMD:C_0402_1005Metric_Pad0.74x0.62mm_HandSolder, F.Cu at (75.7, 84.5)
- added C27: 1uF, Capacitor_SMD:C_0402_1005Metric_Pad0.74x0.62mm_HandSolder, F.Cu at (74.8, 102.0)
- added C33: 680uF, Capacitor_SMD:CP_Elec_10x10, B.Cu at (103.4, 65.6)
- added J18: Sensor power lines, Connector_PinHeader_2.54mm:PinHeader_2x04_P2.54mm_Horizontal, F.Cu at (109.8, 111.8)
- added R3: 5.1K, Resistor_SMD:R_0603_1608Metric, F.Cu at (52.8, 100.4)
- added R4: 5.1K, Resistor_SMD:R_0603_1608Metric, F.Cu at (52.8, 97.5)
- added U4: DFN_XGIQ_TR_WIN, footprints:DFN_XGIQ TR_WIN-M, F.Cu at (66.2, 99.8)
- moved C1 218.2 mm to (47.1, 56.7), turned to 180 degrees
- moved C2 214.6 mm to (50.2, 56.7)
- moved C6 211.4 mm to (47.0, 73.5), turned to 180 degrees
- moved C5 209.1 mm to (50.0, 73.5)
- moved C19 209.1 mm to (46.7, 89.5), turned to 180 degrees
- moved C20 205.9 mm to (49.6, 89.5)
- moved C7 190.7 mm to (70.4, 66.2)
- moved C9 190.5 mm to (70.4, 64.7)
- moved J19 175.7 mm to (94.0, 111.3)
- moved C29 170.2 mm to (89.0, 94.0)
- moved C30 170.0 mm to (89.0, 92.9)
- moved J11 168.3 mm to (45.5, 76.3), turned to 90 degrees
- moved J9 166.3 mm to (45.5, 70.4), turned to 90 degrees
- moved J8 163.0 mm to (45.5, 79.9), turned to 90 degrees
- moved J6 162.6 mm to (45.5, 66.8), turned to 90 degrees
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- renumbered C33 to C1, C37 to C11, C37 to C12, C5 to C14, C3 to C15, C4 to C16, C6 to C17, C7 to C18, C25 to C19, C23 to C2, C27 to C20, C40 to C21, C10 to C22, C21 to C23, C37 to C24, C41 to C25, C10 to C26, C37 to C28, C34 to C29, C9 to C3, C16 to C30, C1 to C31, C2 to C32, C8 to C4, C36 to C5, C32 to C6, C20 to C7, C37 to C8, C30 to C9, D8 to D7, D9 to D8, D7 to D9, J14 to J10, J20 to J12, J8 to J13, J2 to J14, J3 to J15, J19 to J16, J18 to J17, J21 to J19, J10 to J2, J4 to J20, J5 to J21, J9 to J22, J12 to J3, J7 to J4, J6 to J5, J16 to J6, J17 to J7, J15 to J8, J13 to J9, R3 to R1, R6 to R2, R4 to R5, R5 to R6, SW2 to SW1, SW1 to SW2, U4 to U1, U1 to U2, U2 to U3
Connections:
- J15 pad 1: Net-(J1-Pin_10) -> Net-(J3-Pin_1)
- J15 pad 2: Net-(J1-Pin_8) -> Net-(J3-Pin_2)
- J15 pad 25: Net-(J3-Pin_25) -> Net-(J1-Pin_10)
- J15 pad 26: Net-(J3-Pin_26) -> Net-(J1-Pin_8)
- U5 pad 11: Net-(J3-Pin_9) -> Net-(J3-Pin_17)
- U5 pad 12: Net-(J3-Pin_10) -> Net-(J3-Pin_18)
- U5 pad 13: Net-(J3-Pin_11) -> Net-(J3-Pin_15)
- U5 pad 14: Net-(J3-Pin_12) -> Net-(J3-Pin_16)
- U5 pad 17: Net-(J3-Pin_15) -> Net-(J3-Pin_11)
- U5 pad 18: Net-(J3-Pin_16) -> Net-(J3-Pin_12)
- U5 pad 27: Net-(J3-Pin_17) -> Net-(J3-Pin_9)
- U5 pad 28: Net-(J3-Pin_18) -> Net-(J3-Pin_10)
- U5 pad 29: Net-(J3-Pin_19) -> Net-(J3-Pin_7)
- U5 pad 30: Net-(J3-Pin_20) -> Net-(J3-Pin_8)
- U5 pad 31: Net-(J3-Pin_21) -> Net-(J3-Pin_5)
- U5 pad 32: Net-(J3-Pin_22) -> Net-(J3-Pin_6)
- U5 pad 34: Net-(J3-Pin_23) -> Net-(J3-Pin_3)
- U5 pad 35: Net-(J3-Pin_24) -> Net-(J3-Pin_4)
- U5 pad 36: Net-(J3-Pin_25) -> Net-(J3-Pin_1)
- U5 pad 37: Net-(J3-Pin_26) -> Net-(J3-Pin_2)
- U5 pad 4: Net-(J3-Pin_3) -> Net-(J3-Pin_23)
- U5 pad 5: Net-(J3-Pin_4) -> Net-(J3-Pin_24)
- U5 pad 6: Net-(J3-Pin_5) -> Net-(J3-Pin_21)
- U5 pad 7: Net-(J3-Pin_6) -> Net-(J3-Pin_22)
- U5 pad 8: Net-(J3-Pin_7) -> Net-(J3-Pin_19)
- U5 pad 9: Net-(J3-Pin_8) -> Net-(J3-Pin_20)
Routing:
- net +3V3: track 83.8 -> 415.8 mm, vias 0 -> 5
- net +5V: track 8.13 -> 180.6 mm, vias 0 -> 2
- net /SCL: track 0.00 -> 166.2 mm, vias 0 -> 5
- net /SDA: track 0.00 -> 164.1 mm, vias 0 -> 8
- net Net-(J1-Pin_8): track 0.00 -> 106.5 mm
- net Net-(J1-Pin_10): track 0.00 -> 99.9 mm
- net Net-(J1-Pin_36): track 0.00 -> 67.6 mm, vias 0 -> 1
- net Net-(J1-Pin_12): track 0.00 -> 64.9 mm
- net Net-(J1-Pin_11): track 0.00 -> 63.4 mm
- net Net-(J1-Pin_16): track 0.00 -> 61.7 mm, vias 0 -> 1
- net Net-(J1-Pin_13): track 0.00 -> 60.7 mm
- net Net-(J1-Pin_38): track 0.00 -> 58.1 mm, vias 0 -> 1
- net Net-(J1-Pin_40): track 0.00 -> 58.0 mm, vias 0 -> 2
- net Net-(J1-Pin_15): track 0.00 -> 54.2 mm
- net Net-(J1-Pin_35): track 0.00 -> 52.8 mm, vias 0 -> 1
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- added copper zone on F.Cu, net +3V3
- added copper zone on B.Cu, net GND
- added copper zone on F.Cu, net GND
- added copper zone on In1.Cu, net GND
- added copper zone on In2.Cu, net GND
Other:
- board outline added: 117.5 x 73 mm
- copper layers 2 -> 4
- board text added: "Front UsDS"
- board text added: "Rear UsDS"
